File: robot.kicad_sch (KiCad schematic)
At the start: 35 parts, among them J1 Conn_02x06_Top_Bottom, J2 Conn_02x18_Counter_Clockwise, J4 Conn_02x06_Top_Bottom, J6 Conn_02x06_Top_Bottom, M1 SERVO, M4 MOTOR, M5 MOTOR, M6 SERVO, M7 MOTOR, M8 MOTOR, M9 MOTOR, U1 BUCKCONVERTER, U10 SINGLETB9051FTG_MOTOR_DRIVER, U11 ENCODER, U12 MEEN3230_POWER_BOARD, U2 TCS3200, U3 XBEE_DONGLE, U4 SINGLETB9051FTG_MOTOR_DRIVER, U5 ENCODER, U6 SHARPDISTANCE, U7 HALL-EFFECT, U8 SINGLETB9051FTG_MOTOR_DRIVER, U9 ENCODER

Commit message: Schematic Overhaul
Parts:
- removed J1, J4, J6: Conn_02x06_Top_Bottom, symbol Connector_Generic:Conn_02x06_Top_Bottom
- removed J2: Conn_02x18_Counter_Clockwise, symbol Connector_Generic:Conn_02x18_Counter_Clockwise
- removed M8, M9: MOTOR, MOTOR:VIBE-MOTOR-10MM, symbol ME3230:MOTOR
- removed U10, U4, U8: SINGLETB9051FTG_MOTOR_DRIVER, SINGLETB9051FTG_MOTOR_DRIVER:SINGLETB9051FTG, symbol ME3230:SINGLETB9051FTG_MOTOR_DRIVER
- removed U11, U9: ENCODER, ENCODER:ENCODER, symbol ME3230:ENCODER
- added M2, M3: MOTOR, MOTOR:VIBE-MOTOR-10MM, symbol ME3230:MOTOR
- added U5, U6: ENCODER, ENCODER:ENCODER, symbol ME3230:ENCODER
- renumbered M7 to M1, M1 to M7, S1 to S4, U7 to U10, U5 to U4, U1 to U7, U6 to U8, U2 to U9, U3 to W1
Connections:
- net Motors/M1_4: now reaches U4.P1 (GND)
- net Motors/M1_1: now reaches U4.P2 (OUTA)
- net Motors/M1_2: now reaches U4.P3 (OUTB)
- net Motors/M1_3: now reaches U4.P4 (VIN)
- net Motors/M1_6: now reaches M1.+
- net Motors/M1_5: now reaches M1.-
- new net Motors/M2_1: U5.P2 (OUTA)
- new net Motors/M2_2: U5.P3 (OUTB)
- new net Motors/M2_3: U5.P4 (VIN)
- new net Motors/M2_4: U5.P1 (GND)
- new net Motors/M2_5: M2.-
- new net Motors/M2_6: M2.+
- new net Motors/M3_1: U6.P2 (OUTA)
- new net Motors/M3_2: U6.P3 (OUTB)
- new net Motors/M3_3: U6.P4 (VIN)
- new net Motors/M3_4: U6.P1 (GND)
- new net Motors/M3_5: M3.-
- new net Motors/M3_6: M3.+
- no-connect marks 57 -> 46
Other:
- added sheet Motors (motor.kicad_sch)
- note added: "1: White 2: Yellow 3: Blue 4: Green 5: Black 6: Red"
- note added: "Red: Motor+ Black: Motor- Green: GND Blue: Encoder VCC Yellow: Encoder A White: Encoder B"
- note removed: "18-Wide Ribbon Cable to Arduino"
- note removed: "1: PWM 2: Control 1 3: Control 2 4: Current Reading 5: Encoder B 6: Encoder A"
- note removed: "For Motors Red: Power+, Black: Power- Green: GND, Blue: Encoder VCC (5V) Yellow/White: Encoder Outputs"
- note removed: "Logic Power from Buck"
- note removed: "Motors Ground"
- note removed: "Power from Battery"
- title: (none) -> Full Robot Schematic
- moved on the sheet: D4, M1, M4, M5, M6, M7, R1, R2, R3, S1, S2, U10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
