File: schematic/motor.kicad_sch (KiCad schematic)
At the start: 8 parts, among them J1 Conn_02x06_Row_Letter_Last, J2 Conn_02x06_Row_Letter_Last, J3 Conn_02x06_Row_Letter_Last, J4 Screw_Terminal_01x02, J5 Conn_02x18_Row_Letter_Last, U1 SINGLETB9051FTG_MOTOR_DRIVER, U2 SINGLETB9051FTG_MOTOR_DRIVER, U3 SINGLETB9051FTG_MOTOR_DRIVER

Commit message: Full PM7 working
Other:
- note added: "encoder A"
- note added: "encoder B"
Changed lines of the file:
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@@
+		)
+	)
+	(text "encoder B"
+		(exclude_from_sim no)
+		(at 170.18 118.618 0)
+		(effects
+			(font
+				(size 1.27 1.27)
+			)
+		)
+	)
+	(text "encoder A"
+		(exclude_from_sim no)
+		(at 170.18 121.158 0)
+		(effects
+			(font
+				(size 1.27 1.27)
+			)
 		)
 	)
@@
 		)
 	)
+	(text "encoder A"
+		(exclude_from_sim no)
+		(at 170.434 80.01 0)
+		(effects
+			(font
+				(size 1.27 1.27)
+			)
+		)
+	)
 	(text "Yellow"
 		(exclude_from_sim no)
@@
 		(effects
 			(font
+				(size 1.27 1.27)
+			)
+		)
+	)
+	(text "encoder B"
+		(exclude_from_sim no)
+		(at 170.434 77.47 0)
+		(effects
+			(font

Commit message: I don't even know at this point, so much changed
Connections:
- net MC1 renamed MC1_1
- net MC10 renamed MC2_4
- net MC11 renamed MC2_5
- net MC12 renamed MC2_6
- net MC13 renamed MC3_1
- net MC14 renamed MC3_2
- net MC15 renamed MC3_3
- net MC16 renamed MC3_4
- net MC17 renamed MC3_5
- net MC18 renamed MC3_6
- net MC2 renamed MC1_2
- net MC3 renamed MC1_3
- net MC4 renamed MC1_4
- net MC5 renamed MC1_5
- net MC6 renamed MC1_6
- net MC7 renamed MC2_1
- net MC8 renamed MC2_2
- net MC9 renamed MC2_3
Changed lines of the file:
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@@
 		)
 	)
-	(hierarchical_label "MC14"
+	(hierarchical_label "MC3_2"
 		(shape input)
 		(at 27.94 68.58 180)
@@
 		)
 	)
-	(hierarchical_label "MC1"
+	(hierarchical_label "MC1_1"
 		(shape input)
 		(at 27.94 35.56 180)
@@
 		)
 	)
-	(hierarchical_label "MC13"
+	(hierarchical_label "MC3_1"
 		(shape input)
 		(at 27.94 66.04 180)
@@
 		)
 	)
-	(hierarchical_label "MC10"
+	(hierarchical_label "MC2_4"
 		(shape input)
 		(at 27.94 58.42 180)
@@
 		)
 	)
-	(hierarchical_label "MC16"
+	(hierarchical_label "MC3_4"
 		(shape input)
 		(at 27.94 73.66 180)
@@
 		)
 	)
-	(hierarchical_label "MC11"
+	(hierarchical_label "MC2_5"
 		(shape input)
 		(at 27.94 60.96 180)
@@
 		)
 	)
-	(hierarchical_label "MC9"
+	(hierarchical_label "MC2_3"
 		(shape input)
 		(at 27.94 55.88 180)
@@
 		)
 	)
-	(hierarchical_label "MC3"
+	(hierarchical_label "MC1_3"
 		(shape input)
 		(at 27.94 40.64 180)
@@
 		)
 	)
-	(hierarchical_label "MC7"
+	(hierarchical_label "MC2_1"
 		(shape input)
 		(at 27.94 50.8 180)
@@
 		)
 	)
-	(hierarchical_label "MC5"
+	(hierarchical_label "MC1_5"
 		(shape input)
 		(at 27.94 45.72 180)
@@
 		)
 	)
-	(hierarchical_label "MC8"
+	(hierarchical_label "MC2_2"
 		(shape input)
 		(at 27.94 53.34 180)
@@
 		)
 	)
-	(hierarchical_label "MC12"
+	(hierarchical_label "MC2_6"
 		(shape input)
 		(at 27.94 63.5 180)
@@
 		)
 	)
-	(hierarchical_label "MC6"
+	(hierarchical_label "MC1_6"
 		(shape input)
 		(at 27.94 48.26 180)
@@
 		)
 	)
-	(hierarchical_label "MC15"
+	(hierarchical_label "MC3_3"
 		(shape input)
 		(at 27.94 71.12 180)
@@
 		)
 	)
-	(hierarchical_label "MC4"
+	(hierarchical_label "MC1_4"
 		(shape input)
 		(at 27.94 43.18 180)
@@
 		)
 	)
-	(hierarchical_label "MC17"
+	(hierarchical_label "MC3_5"
 		(shape input)
 		(at 27.94 76.2 180)
@@
 		)
 	)
-	(hierarchical_label "MC2"
+	(hierarchical_label "MC1_2"
 		(shape input)
 		(at 27.94 38.1 180)
@@
 		)
 	)
-	(hierarchical_label "MC18"
+	(hierarchical_label "MC3_6"
 		(shape input)
 		(at 27.94 78.74 180)
